File: PCB/LAWO_ESP32/LAWO_ESP32.sch (KiCad schematic (older format))
At the start: 54 parts, among them J1 Barrel_Jack, J2 Screw_Terminal_01x06, P1 MATRIX, P2 MUX, Q1 BC547, Q2 IRF740, SW1 T1, SW2 T2, U1 L7805, U2 LM317T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

Commit message: update
Connections:
- net MCP_RESET: now also P2.11 (P11)
- net SCL: now also P2.13 (P13)
- net SDA: now also P2.15 (P15)
- no-connect marks 29 -> 26
Changed lines of the file:
@@
 NoConn ~ 10590 1870
 NoConn ~ 10590 1970
-NoConn ~ 10090 1670
-NoConn ~ 10090 1770
-NoConn ~ 10090 1870
 NoConn ~ 10090 1970
 NoConn ~ 14050 7100
@@
 Wire Notes Line
 	7890 7910 8530 7910
+Text Notes 7870 8210 0    60   ~ 0
+ Low\n Side\n(Reset)
+Text Notes 8280 8210 0    60   ~ 0
+High\nSide\n(Set)
 Wire Bus Line
 	4350 6620 4350 8250
@@
 Wire Bus Line
 	12040 6600 12040 8260
-Text Notes 7870 8210 0    60   ~ 0
- Low\n Side\n(Reset)
-Text Notes 8280 8210 0    60   ~ 0
-High\nSide\n(Set)
+Text Label 10090 1670 2    60   ~ 0
+MCP_RESET
+Text Label 10090 1770 2    60   ~ 0
+SCL
+Text Label 10090 1870 2    60   ~ 0
+SDA
 $EndSCHEMATC
