File: PCB/LAWO_ESP32/LAWO_ESP32.kicad_pcb (KiCad board)
At the start: 2 copper layers, 100 x 100 mm, 54 parts, among them J1 Barrel_Jack, J2 Screw_Terminal_01x06, P1 MATRIX, P2 MUX, Q1 BC547, Q2 IRF740, SW1 T1, SW2 T2, U1 L7805, U2 LM317T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

Commit message: update
Connections:
- P2 pad 11: Net-(P2-Pad11) -> /MCP_RESET
- P2 pad 13: Net-(P2-Pad13) -> /SCL
- P2 pad 15: Net-(P2-Pad15) -> /SDA
Routing:
- net /MCP_RESET: track 72.9 -> 174.2 mm
- net /SCL: track 96.4 -> 184.1 mm
- net /SDA: track 94.3 -> 178.9 mm
- net GND: track 390.0 -> 363.3 mm
- net +5V: track 311.0 -> 310.3 mm, vias 3 -> 5

Commit message: update
Parts:
- moved R18 10.5 mm to (77.5, 26.4), turned to 0 degrees
Routing:
- net GND: track 363.3 -> 342.0 mm, vias 3 -> 14
- net /SCL: track 184.1 -> 182.2 mm
- net +5V: track 310.3 -> 311.2 mm
Other:
- board text added: "+5V"
- board text added: "COL A0"
- board text added: "COL A1"
- board text added: "COL A2"
- board text added: "COL A3"
- board text added: "COL A4"
- board text added: "D"
- board text added: "E1"
- board text added: "E2"
- board text added: "E3"
- board text added: "E4"
- board text added: "E5"
- board text added: "GND"
- board text added: "IN"
- board text added: "LED D2"
- board text added: "LED D3"
- board text added: "MCP RESET"
- board text added: "MCP23017"
- board text added: "NC"
- board text added: "SCL"
- board text added: "SDA"
- board text added: "SW1"
- board text added: "SW2"
- board text added: "UDN2981A"
- board text added: "ULN2803A"
- board text added: "ext. LED"
